File: chaudiere/poisson2.kicad_pcb (KiCad board)
At the start: 2 copper layers, 100 x 100 mm, 74 parts, among them J1 Conn_02x12_Top_Bottom, J10 Conn_01x02_Female, J11 Screw_Terminal_01x02, J12 Conn_01x02_Female, J13 Screw_Terminal_01x02, J14 Conn_01x02_Female, J15 Screw_Terminal_01x02, J16 Conn_01x02_Female, J17 Screw_Terminal_01x02, J18 Conn_01x02_Female, J19 Conn_01x02_Female, J2 Conn_01x02_Male, J20 Conn_01x02_Female, J21 Conn_01x02_Female, J22 Screw_Terminal_01x02, J23 Screw_Terminal_01x02, J24 Screw_Terminal_01x02, J25 Conn_01x02_Female, J26 Conn_01x02_Female, J27 Conn_01x02_Female, J28 Conn_01x02_Female, J3 Conn_01x02_Female, J4 Conn_01x02_Female, J5 Conn_01x02_Female, J6 Conn_01x02_Female, J7 Conn_01x02_Female, J8 Conn_02x05_Counter_Clockwise, J9 Conn_02x05_Top_Bottom, Q1 BC548, Q2 BC548, Q3 BC548, Q4 BC548, Q5 BC548, U2 ESP8266EX-NODEMCU-FRED-chaudi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

Commit message: GFFH
Parts:
-  : renamed from REF** (x6)
Connections:
-   pad 1: (no net) -> +3V3 (x3)
Routing:
- net +3V3: track 397.8 -> 441.2 mm
- net GND: track 1373.8 -> 1382.3 mm
Other:
- board text added: "+"
- board text added: "-"
- board text added: "D+"
- board text added: "D-"
