File: chaudiere3/poisson2.sch (KiCad schematic (older format))
At the start: 58 parts, among them J1 Conn_02x12_Top_Bottom, J10 Conn_01x02_Female, J11 Screw_Terminal_01x02, J12 Conn_01x02_Female, J13 Screw_Terminal_01x02, J14 Conn_01x02_Female, J15 Screw_Terminal_01x02, J16 Conn_01x02_Female, J17 Screw_Terminal_01x02, J18 Conn_01x02_Female, J19 Conn_01x02_Female, J2 Conn_01x02_Male, J20 Conn_01x02_Female, J21 Conn_01x02_Female, J22 Screw_Terminal_01x02, J23 Screw_Terminal_01x02, J24 Screw_Terminal_01x02, J25 Conn_01x02_Female, J3 Conn_01x02_Female, J4 Conn_01x02_Female, J5 Conn_01x02_Female, J6 Conn_01x02_Female, J7 Conn_01x02_Female, J8 Conn_02x05_Counter_Clockwise, J9 Conn_02x05_Top_Bottom, Q1 BC548, Q2 BC548, Q3 BC548, Q4 BC548, Q5 BC548, U2 ESP8266EX-NODEMCU-FRED-chaudi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

Commit message: cau
Parts:
- added C1: CP, Capacitor_THT:CP_Radial_D5.0mm_P2.50mm, symbol Device:CP
- added J26, J27, J28: Conn_01x02_Female, Connector_PinHeader_2.54mm:PinHeader_1x02_P2.54mm_Vertical, symbol Connector:Conn_01x02_Female
- J1: footprint atx:atx_couder -> atx:atx_couder_femelle
Connections:
- net +3V3: now also C1.1
- net GND: now also C1.2, J26.2 (Pin_2), J27.2 (Pin_2), J28.2 (Pin_2)
- net at U2.21 (Gpio13): now also J27.1 (Pin_1)
- net at U2.30 (Gpio16): now also J26.1 (Pin_1), J28.1 (Pin_1)
Changed lines of the file:
@@
 F 0 "J1" H 9750 10017 50  0000 C CNN
 F 1 "Conn_02x12_Top_Bottom" H 9750 9926 50  0000 C CNN
-F 2 "atx:atx_couder" H 9700 9300 50  0001 C CNN
+F 2 "atx:atx_couder_femelle" H 9700 9300 50  0001 C CNN
 F 3 "~" H 9700 9300 50  0001 C CNN
 	1    9700 9300
@@
 Wire Wire Line
 	8650 9400 9500 9400
+Wire Wire Line
+	5700 2450 5700 3350
+Wire Wire Line
+	5700 3350 5350 3350
+Wire Wire Line
+	5350 3350 5350 3200
+$Comp
+L Connector:Conn_01x02_Female J27
+U 1 1 5DE62A45
+P 7500 2400
+F 0 "J27" H 7528 2376 50  0000 L CNN
+F 1 "Conn_01x02_Female" H 7528 2285 50  0000 L CNN
+F 2 "Connector_PinHeader_2.54mm:PinHeader_1x02_P2.54mm_Vertical" H 7500 2400 50  0001 C CNN
+F 3 "~" H 7500 2400 50  0001 C CNN
+	1    7500 2400
+	1    0    0    -1
+$EndComp
+$Comp
+L power:GND #PWR0121
+U 1 1 5DE62A50
+P 7300 2550
+F 0 "#PWR0121" H 7300 2300 50  0001 C CNN
+F 1 "GND" H 7305 2377 50  0000 C CNN
+F 2 "" H 7300 2550 50  0001 C CNN
+F 3 "" H 7300 2550 50  0001 C CNN
+	1    7300 2550
+	1    0    0    -1
+$EndComp
+Wire Wire Line
+	7300 2500 7300 2550
+Wire Wire Line
+	7150 2400 7150 2900
+Wire Wire Line
+	7150 2900 5350 2900
+Wire Wire Line
+	7150 2400 7300 2400
+$Comp
+L Connector:Conn_01x02_Female J28
+U 1 1 5DE98A8F
+P 6050 2450
+F 0 "J28" H 6078 2426 50  0000 L CNN
+F 1 "Conn_01x02_Female" H 6078 2335 50  0000 L CNN
+F 2 "Connector_PinHeader_2.54mm:PinHeader_1x02_P2.54mm_Vertical" H 6050 2450 50  0001 C CNN
+F 3 "~" H 6050 2450 50  0001 C CNN
+	1    6050 2450
+	1    0    0    -1
+$EndComp
+$Comp
+L power:GND #PWR0120
+U 1 1 5DE98A99
+P 5850 2600
+F 0 "#PWR0120" H 5850 2350 50  0001 C CNN
+F 1 "GND" H 5855 2427 50  0000 C CNN
+F 2 "" H 5850 2600 50  0001 C CNN
+F 3 "" H 5850 2600 50  0001 C CNN
+	1    5850 2600
+	1    0    0    -1
+$EndComp
+Wire Wire Line
+	5850 2550 5850 2600
+Wire Wire Line
+	5700 2450 5850 2450
+$Comp
+L Connector:Conn_01x02_Female J26
+U 1 1 5DEA936F
+P 6050 2200
+F 0 "J26" H 6078 2176 50  0000 L CNN
+F 1 "Conn_01x02_Female" H 6078 2085 50  0000 L CNN
+F 2 "Connector_PinHeader_2.54mm:PinHeader_1x02_P2.54mm_Vertical" H 6050 2200 50  0001 C CNN
+F 3 "~" H 6050 2200 50  0001 C CNN
+	1    6050 2200
+	1    0    0    -1
+$EndComp
+$Comp
+L power:GND #PWR0122
+U 1 1 5DEA9379
+P 5850 2350
+F 0 "#PWR0122" H 5850 2100 50  0001 C CNN
+F 1 "GND" H 5855 2177 50  0000 C CNN
+F 2 "" H 5850 2350 50  0001 C CNN
+F 3 "" H 5850 2350 50  0001 C CNN
+	1    5850 2350
+	1    0    0    -1
+$EndComp
+Wire Wire Line
+	5850 2300 5850 2350
+Wire Wire Line
+	5700 2200 5850 2200
+Wire Wire Line
+	5700 2200 5700 2450
+Connection ~ 5700 2450
+$Comp
+L Device:CP C1
+U 1 1 5DED850E
+P 11050 8750
+F 0 "C1" H 11168 8796 50  0000 L CNN
+F 1 "CP" H 11168 8705 50  0000 L CNN
+F 2 "Capacitor_THT:CP_Radial_D5.0mm_P2.50mm" H 11088 8600 50  0001 C CNN
+F 3 "~" H 11050 8750 50  0001 C CNN
+	1    11050 8750
+	1    0    0    -1
+$EndComp
+Wire Wire Line
+	11050 8600 10750 8600
+Wire Wire Line
+	10750 8600 10750 8800
+Wire Wire Line
+	10750 8800 10550 8800
+Wire Wire Line
+	11050 8900 11050 9000
+Wire Wire Line
+	11050 9000 10200 9000
 $EndSCHEMATC
